File: schematics/beltdrive/beltdrive.sch (KiCad schematic (older format))
At the start: 2 parts

Commit message: finished rear motormount💦
Parts:
- removed A?: Arduino_UNO_R3, Module:Arduino_UNO_R3, symbol MCU_Module:Arduino_UNO_R3
- removed J?: Raspberry_Pi_2_3, symbol Connector:Raspberry_Pi_2_3
- added .?: ESC, symbol generic_symbols:ESC
- added A?: Arduino_Nano_v3.x, Module:Arduino_Nano, symbol MCU_Module:Arduino_Nano_v3.x
Connections:
- new net +5V: A?.27 (+5V)
Changed lines of the file:
@@
 EESchema Schematic File Version 4
+LIBS:beltdrive-cache
 EELAYER 29 0
 EELAYER END
@@
 $EndDescr
 $Comp
-L Connector:Raspberry_Pi_2_3 J?
-U 1 1 5CAC6586
-P 3800 4950
-F 0 "J?" H 3800 6431 50  0000 C CNN
-F 1 "Raspberry_Pi_2_3" H 3800 6340 50  0000 C CNN
-F 2 "" H 3800 4950 50  0001 C CNN
-F 3 "https://www.raspberrypi.org/documentation/hardware/raspberrypi/schematics/rpi_SCH_3bplus_1p0_reduced.pdf" H 3800 4950 50  0001 C CNN
-	1    3800 4950
+L MCU_Module:Arduino_Nano_v3.x A?
+U 1 1 5CACB588
+P 3250 2350
+F 0 "A?" H 3250 1261 50  0000 C CNN
+F 1 "Arduino_Nano_v3.x" H 3250 1170 50  0000 C CNN
+F 2 "Module:Arduino_Nano" H 3400 1400 50  0001 L CNN
+F 3 "http://www.mouser.com/pdfdocs/Gravitech_Arduino_Nano3_0.pdf" H 3250 1350 50  0001 C CNN
+	1    3250 2350
 	1    0    0    -1
 $EndComp
 $Comp
-L MCU_Module:Arduino_UNO_R3 A?
-U 1 1 5CACCBD7
-P 5700 2650
-F 0 "A?" H 5700 3831 50  0000 C CNN
-F 1 "Arduino_UNO_R3" H 5700 3740 50  0000 C CNN
-F 2 "Module:Arduino_UNO_R3" H 5850 1600 50  0001 L CNN
-F 3 "https://www.arduino.cc/en/Main/arduinoBoardUno" H 5500 3700 50  0001 C CNN
-	1    5700 2650
+L power:+5V #PWR?
+U 1 1 5CAD2A4D
+P 3450 900
+F 0 "#PWR?" H 3450 750 50  0001 C CNN
+F 1 "+5V" H 3465 1073 50  0000 C CNN
+F 2 "" H 3450 900 50  0001 C CNN
+F 3 "" H 3450 900 50  0001 C CNN
+	1    3450 900
 	1    0    0    -1
 $EndComp
+Wire Wire Line
+	3450 900  3450 1350
+$Comp
+L generic_symbols:ESC .?
+U 1 1 5CAD71D4
+P 5800 2100
+F 0 ".?" H 5800 2100 50  0001 C CNN
+F 1 "ESC" H 4681 1925 50  0000 R CNN
+F 2 "" H 5800 2100 50  0001 C CNN
+F 3 "" H 5800 2100 50  0001 C CNN
+	1    5800 2100
+	1    0    0    -1
+$EndComp
